File: src/counterspell.kicad_sch (KiCad schematic)
At the start: 9 parts, among them SW1 SW_Push

Commit message: important
Connections:
- net at D1.2 (A): now also C1.1, D2.2 (A), D3.2 (A), SW1.2; no longer R2.1
- net at R1.1: now also D3.1 (K); no longer D3.2 (A)
- net at R3.1: now also D2.1 (K); no longer D2.2 (A)
- new net: D1.1 (K), R2.1
Other:
- moved on the sheet: D1
Changed lines of the file:
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@@
+	)
+	(junction
+		(at 77.47 64.77)
+		(diameter 0)
+		(color 0 0 0 0)
+	)
+	(junction
+		(at 77.47 58.42)
+		(diameter 0)
+		(color 0 0 0 0)
 	)
 	(junction
@@
 	)
 	(junction
-		(at 77.47 64.77)
-		(diameter 0)
-		(color 0 0 0 0)
-	)
-	(junction
-		(at 77.47 58.42)
-		(diameter 0)
-		(color 0 0 0 0)
-	)
-	(junction
 		(at 95.25 73.66)
 		(diameter 0)
@@
 	(wire
 		(pts
+			(xy 77.47 58.42) (xy 77.47 64.77)
+		)
+		(stroke
+			(width 0)
+			(type default)
+		)
+	)
+	(wire
+		(pts
+			(xy 63.5 50.8) (xy 76.2 50.8)
+		)
+		(stroke
+			(width 0)
+			(type default)
+		)
+	)
+	(wire
+		(pts
+			(xy 83.82 50.8) (xy 95.25 50.8)
+		)
+		(stroke
+			(width 0)
+			(type default)
+		)
+	)
+	(wire
+		(pts
 			(xy 77.47 64.77) (xy 77.47 73.66)
-		)
-		(stroke
-			(width 0)
-			(type default)
-		)
-	)
-	(wire
-		(pts
-			(xy 63.5 50.8) (xy 76.2 50.8)
-		)
-		(stroke
-			(width 0)
-			(type default)
-		)
-	)
-	(wire
-		(pts
-			(xy 83.82 50.8) (xy 95.25 50.8)
-		)
-		(stroke
-			(width 0)
-			(type default)
-		)
-	)
-	(wire
-		(pts
-			(xy 77.47 58.42) (xy 77.47 64.77)
 		)
 		(stroke
@@
 	(symbol
 		(lib_id "Device:LED")
-		(at 81.28 58.42 0)
+		(at 81.28 58.42 180)
 		(unit 1)
 		(exclude_from_sim no)
@@
 		(dnp no)
 		(property "Reference" "D3"
-			(at 80.518 68.834 0)
-			(effects
-				(font
-					(size 1.27 1.27)
-				)
+			(at 82.042 48.006 0)
+			(effects
+				(font
+					(size 1.27 1.27)
+				)
+				(hide yes)
 			)
 		)
 		(property "Value" "LED"
-			(at 80.518 71.374 0)
-			(effects
-				(font
-					(size 1.27 1.27)
-				)
+			(at 82.042 45.466 0)
+			(effects
+				(font
+					(size 1.27 1.27)
+				)
+				(hide yes)
 			)
 		)
@@
 	(symbol
 		(lib_id "Device:LED")
-		(at 81.28 64.77 0)
+		(at 81.28 64.77 180)
 		(unit 1)
 		(exclude_from_sim no)
@@
 		(fields_autoplaced yes)
 		(property "Reference" "D1"
-			(at 79.6925 58.42 0)
+			(at 82.8675 57.15 0)
 			(effects
 				(font
@@
 		)
 		(property "Value" "LED"
-			(at 79.6925 60.96 0)
+			(at 82.8675 59.69 0)
 			(effects
 				(font
@@
 	(symbol
 		(lib_id "Device:LED")
-		(at 81.28 73.66 0)
+		(at 81.28 73.66 180)
 		(unit 1)
 		(exclude_from_sim no)
@@
 		(dnp no)
 		(property "Reference" "D2"
-			(at 83.82 62.23 0)
-			(effects
-				(font
-					(size 1.27 1.27)
-				)
+			(at 78.74 85.09 0)
+			(effects
+				(font
+					(size 1.27 1.27)
+				)
+				(hide yes)
 			)
 		)
 		(property "Value" "LED"
-			(at 84.328 64.262 0)
-			(effects
-				(font
-					(size 1.27 1.27)
-				)
-			)
-		)
+			(at 78.232 83.058 0)
+			(effects
+				(font
+					(size 1.27 1.27)
+				)
+				(hide yes)
+			)
+		)
